File: kicad-test1/kicad-test1.sch (KiCad schematic (older format))
At the start: 3 parts

Commit message: Jo
Parts:
- D1: Spice_Model Dled_test -> LED
- gave numbers to parts that had none: 1
Changed lines of the file:
@@
 F 3 "~" H 5150 2500 50  0001 C CNN
 F 4 "D" H 5150 2500 50  0001 C CNN "Spice_Primitive"
-F 5 "Dled_test" H 5150 2500 50  0001 C CNN "Spice_Model"
+F 5 "LED" H 5150 2500 50  0001 C CNN "Spice_Model"
 F 6 "Y" H 5150 2500 50  0001 C CNN "Spice_Netlist_Enabled"
 F 7 "led.lib" H 5150 2500 50  0001 C CNN "Spice_Lib_File"
@@
 This is a test
 $Comp
-L pspice:VSOURCE V?
+L pspice:VSOURCE V1
 U 1 1 609FF3B0
 P 2750 1950
-F 0 "V?" H 2978 1996 50  0000 L CNN
+F 0 "V1" H 2978 1996 50  0000 L CNN
 F 1 "5" H 2978 1905 50  0000 L CNN
 F 2 "" H 2750 1950 50  0001 C CNN
@@
 $EndComp
 $Comp
-L power:VCC #PWR?
+L power:VCC #PWR0101
 U 1 1 60A0120A
 P 2750 2250
-F 0 "#PWR?" H 2750 2100 50  0001 C CNN
+F 0 "#PWR0101" H 2750 2100 50  0001 C CNN
 F 1 "VCC" H 2765 2423 50  0000 C CNN
 F 2 "" H 2750 2250 50  0001 C CNN
@@
 $EndComp
 $Comp
-L power:GND #PWR?
+L power:GND #PWR0102
 U 1 1 60A027CE
 P 2750 1650
-F 0 "#PWR?" H 2750 1400 50  0001 C CNN
+F 0 "#PWR0102" H 2750 1400 50  0001 C CNN
 F 1 "GND" H 2755 1477 50  0000 C CNN
 F 2 "" H 2750 1650 50  0001 C CNN
